File: SynchGaze_Motor_Control/BLDC_Driver.kicad_sch (KiCad schematic)
At the start: 18 parts, among them M601 MOT, U601 MCT8315A1VRGFR

Commit message: rev 1.1
Parts:
- removed R601: 0R, Resistor_SMD:R_0402_1005Metric, symbol Device:R_Small
- added C609: 1u/25V, Capacitor_SMD:C_0402_1005Metric, symbol Device:C_Small
- added R605: 5.1k, Resistor_SMD:R_0402_1005Metric, symbol Device:R_Small
- C601: value 47n -> 47n/25V
- C602, C605, C606: value 1u -> 1u/25V
- C603: value 100n -> 100n/16V
- C604, C608: value 10u -> 10u/25V
- C607: value 10u -> 10u/10V; now fitted; now in the parts list
- L601: now fitted; now in the parts list
Connections:
- net +3V3 is gone; now on net AVDD: R604.1
- net DRV_DRVOFF is gone; now on net GND: U601.21 (DRVOFF)
- net GND: now also C609.2
- net AVDD: now reaches U601.27 (AVDD)
- net AVDD: now also C609.1, R605.1
- net at U601.29 (FG): now also R605.2
- no-connect marks 8 -> 6
Other:
- note removed: "BUCK_CL=1b"
- note removed: "BUCK_PS_DIS=1b"
- note removed: "BUCK_SEL=0h"
- note removed: "NOTE 1"
- note removed: "NOTE 1 Wewnętrzny DVDD LDO wytwarza 1.5V do zasilania logiki. Napięcie Vindvdd jest napięciem branym z pinu FB_BK. Jeżeli rezystor terminujący R307 jest obsadzony, wtedy na pin FB_BK wprowadzone napięcie systemowe 3.3V, nieobsadzony - osadzić L301 i C310. W obu przypadkach odnieść się do datasheet układu i zmienić konfiguracje w pamięci układu."
- note removed: "red"
- moved on the sheet: C603, C604, C605, C606, C608, D601, JP601, R602, R603, R604
