File: SynchGaze_Motor_Control/MCU.kicad_sch (KiCad schematic)
At the start: 48 parts, among them J201 USB4105-GF-A, J202 Molex_0530470810, J203 SWD, J204 Antena connector, SW201 EN, SW202 BOOT, U201 W25Q16JVZPIQ, U202 ESP32C3, U203 USBLC6-2SC6, U204 STM32G4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

Commit message: rev 1.1
Parts:
- removed J203: SWD, A1001WV-S-6P:A1001WV-S-6P, symbol Connector_Generic:Conn_01x06
- added D201: STAT_ESP_Y, LED_SMD:LED_0603_1608Metric, symbol Device:LED
- added D202: STAT_STM_Y, LED_SMD:LED_0603_1608Metric, symbol Device:LED
- added J203: STM32_SWD, PogoPin:PogoConnector, symbol PogoPin:PogoConnector
- added R212, R213, R216, R217: 5.1k, Resistor_SMD:R_0402_1005Metric, symbol Device:R_Small
- added R214, R215: 1k, Resistor_SMD:R_0402_1005Metric, symbol Device:R_Small
- added TP201: FSPI_CLK_TP, TEST_POINT:test_point_SMD_0.5mm, symbol Connector:TestPoint
- added TP202: FSPI_Q_TP, TEST_POINT:test_point_SMD_0.5mm, symbol Connector:TestPoint
- added TP203: FSPI_D_TP, TEST_POINT:test_point_SMD_0.5mm, symbol Connector:TestPoint
- added TP204: IMU_NCS_TP, TEST_POINT:test_point_SMD_0.5mm, symbol Connector:TestPoint
- added TP205: INT2_ACC_TP, TEST_POINT:test_point_SMD_0.5mm, symbol Connector:TestPoint
- added TP206: INT1_GYR_TP, TEST_POINT:test_point_SMD_0.5mm, symbol Connector:TestPoint
- added TP207, TP208: GND, TEST_POINT:test_point_THT 0.7mm, symbol Connector:TestPoint
- added TP209: BOOT, TEST_POINT:test_point_SMD_two_pad_1mm, symbol Connector:TestPoint_2Pole
- C201, C204, C205, C206, C207, C209, C215, C216, C217, C218, C219, C223: value 100n -> 100n/16V
- C202, C203, C208, C210, C220: value 10u -> 10u/10V
- C211, C212: value 3p3 -> 3p3/50V
- C213, C214: value 12p -> 12p/50V
- C221, C222: value 20p -> 20p/16V
- J202: value Molex_0530470810 -> AMPHENOL_75869-132LF; footprint Molex_0530470810:MOLEX_0530470810 -> AMPHENOL_75869-132LF:AMPHENOL_75869-132LF; Manufacturer Molex -> AMPHENOL; TME https://www.tme.eu/pl/details/mx-53047-0810/zlacza-sygnalow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 -> https://www.tme.eu/pl/details/75869-132lf/zlacza-idc/amphen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
Connections:
- net DRVP_DRVOFF is gone; now on net DRVP_ALARM: U204.20 (PA10)
- net +3V3: now also J203.1 (VIN), R212.2, R213.2, R214.2, R215.2, R216.2
- net DRVP_ALARM: no longer U204.31 (PB8-BOOT0)
- net ESP_FSPI_CLK: now also TP201.1
- net ESP_FSPI_D: now also U204.12 (PA7), TP203.1; no longer U204.11 (PA6)
- net ESP_FSPI_NSS: now also R216.1
- net ESP_FSPI_Q: now also U204.11 (PA6), R212.1, TP202.1; no longer U204.12 (PA7)
- net ESP_IMU_NCS: now also TP204.1
- net ESP_SPI_CLK: now also U201.6 (CLK); no longer U201.5 (DI(IO0))
- net ESP_SPI_DI: now also U201.5 (DI(IO0)); no longer U201.2 (DO(IO1))
- net ESP_SPI_DO: now also U201.2 (DO(IO1)); no longer U201.6 (CLK)
- net GND: now also J203.6 (GND), R217.1, TP207.1, TP208.1
- net STM_SWCLK: now also J203.3 (SWCLK)
- net STM_SWDIO: now also J203.2 (SWDIO)
- net STM_SWO: now also J203.4 (SWO)
- net DRVR_DRVOFF/NRST renamed STM_NRST
- net STM_NRST: now also J203.5 (~{RST}), R213.1
- net DRVY_DRVOFF renamed STM_STAT
- net STM_STAT: now also D202.1 (K)
- net ESP_GPIO1 renamed ESP_INT1_GYR
- net ESP_INT1_GYR: now also J202.8 (Pin_8), TP206.1
- net ESP_GPIO10 renamed ESP_STAT
- net ESP_STAT: now also D201.1 (K)
- net ESP_INTER_ACC renamed ESP_INT2_ACC
- net ESP_INT2_ACC: now also TP205.1
- net ESP_INTER_GYR/BOOT renamed ESP_BOOT
- net ESP_BOOT: no longer J202.8 (Pin_8)
- net ESP_UART_RX: no longer names the net of U202.27 (U0RXD)
- net ESP_UART_TX: no longer names the net of U202.28 (U0TXD)
- new net: D202.2 (A), R215.1
- new net: R217.2, TP209.1
- new net: TP209.2, U204.31 (PB8-BOOT0)
- new net: D201.2 (A), R214.1
- no-connect marks 9 -> 7
Other:
- sheet BLDC Driver P ports: added none; removed DRV_DRVOFF
- sheet BLDC Driver R ports: added none; removed DRV_DRVOFF
- sheet BLDC Driver Y ports: added none; removed DRV_DRVOFF
- note added: "BOOT pullup - bootloader BOOT pulldown - normal"
- note removed: "IMU na przewodzie - płytka do zrobienia"
- note removed: "decap cap"
- moved on the sheet: C201, C202, C203, C204, C205, C206, C207, C208, C209, C210, C211, C212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
