File: SynchGaze_Motor_Control/Power.kicad_sch (KiCad schematic)
At the start: 20 parts, among them J402 Input 12V, Q401 SI2347DS, Q402 SI2347DS, U401 TPS62142RGTR

Commit message: rev 1.1
Parts:
- C401, C403, C404: value 10u -> 10u/25V
- C402: value 3.3n -> 3.3n/25V
- D401: value 3V3 -> 3V3_G; Manufacturer Lite-On -> Wurth Elektronik; Manufacturer Part Number LTST-C190GKT -> 150060GS55040; Mouser https://www.mouser.pl/ProductDetail/Lite-On/LTST-C190GKT?qs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 -> https://www.mouser.pl/ProductDetail/Wurth-Elektronik/150060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
- D402: value VIN -> VIN_G; Manufacturer Lite-On -> Wurth Elektronik; Manufacturer Part Number LTST-C190GKT -> 150060GS55040; Mouser https://www.mouser.pl/ProductDetail/Lite-On/LTST-C190GKT?qs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 -> https://www.mouser.pl/ProductDetail/Wurth-Elektronik/150060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
Other:
- note removed: "green"
- moved on the sheet: C402, C404, D401, R401
