File: SynchGaze_Motor_Control/SynchGaze_Motor_Control.kicad_pcb (KiCad board)
At the start: 4 copper layers, 65 x 60 mm, 126 parts, among them J201 USB4105-GF-A, J202 Molex_0530470810, J203 SWD, J204 Antena connector, J402 Input 12V, M301 MOT, M501 MOT, M601 MOT, Q401 SI2347DS, Q402 SI2347DS, SW201 EN, SW202 BOOT, U201 W25Q16JVZPIQ, U202 ESP32C3, U203 USBLC6-2SC6, U204 STM32G4, U301 MCT8315A1VRGFR, U401 TPS62142RGTR, U501 MCT8315A1VRGFR, U601 MCT8315A1VRGFR, X201 XRCGB40M000F4M02R0, X202 830108208209

Commit message: rev 1.1
Parts:
- removed R301, R501, R601: 0R, Resistor_SMD:R_0402_1005Metric
- added C309: 1u/25V, Capacitor_SMD:C_0402_1005Metric, F.Cu at (48.3, 130.9)
- added C509: 1u/25V, Capacitor_SMD:C_0402_1005Metric, F.Cu at (85.3, 130.6)
- added C609: 1u/25V, Capacitor_SMD:C_0402_1005Metric, F.Cu at (66.8, 130.5)
- added D201: STAT_ESP_Y, LED_SMD:LED_0603_1608Metric, F.Cu at (33.0, 98.1)
- added D202: STAT_STM_Y, LED_SMD:LED_0603_1608Metric, F.Cu at (33.0, 99.7)
- added R212: 5.1k, Resistor_SMD:R_0402_1005Metric, F.Cu at (68.9, 107.0)
- added R213: 5.1k, Resistor_SMD:R_0402_1005Metric, F.Cu at (69.5, 113.1)
- added R214: 1k, Resistor_SMD:R_0402_1005Metric, F.Cu at (30.4, 98.1)
- added R215: 1k, Resistor_SMD:R_0402_1005Metric, F.Cu at (30.4, 99.7)
- added R216: 5.1k, Resistor_SMD:R_0402_1005Metric, F.Cu at (71.0, 109.0)
- added R217: 5.1k, Resistor_SMD:R_0402_1005Metric, F.Cu at (65.7, 119.9)
- added R305: 5.1k, Resistor_SMD:R_0402_1005Metric, F.Cu at (48.3, 128.9)
- added R505: 5.1k, Resistor_SMD:R_0402_1005Metric, F.Cu at (85.3, 128.7)
- added R605: 5.1k, Resistor_SMD:R_0402_1005Metric, F.Cu at (66.8, 128.5)
- added TP201: FSPI_CLK_TP, TEST_POINT:test_point_SMD_0.5mm, F.Cu at (80.5, 112.6)
- added TP202: FSPI_Q_TP, TEST_POINT:test_point_SMD_0.5mm, F.Cu at (81.4, 111.9)
- added TP203: FSPI_D_TP, TEST_POINT:test_point_SMD_0.5mm, F.Cu at (81.4, 113.3)
- added TP204: IMU_NCS_TP, TEST_POINT:test_point_SMD_0.5mm, F.Cu at (80.5, 114.1)
- added TP205: INT2_ACC_TP, TEST_POINT:test_point_SMD_0.5mm, F.Cu at (81.4, 114.9)
- added TP206: INT1_GYR_TP, TEST_POINT:test_point_SMD_0.5mm, F.Cu at (80.5, 115.6)
- added TP207: GND, TEST_POINT:test_point_THT 0.7mm, F.Cu at (81.6, 116.5)
- added TP208: GND, TEST_POINT:test_point_THT 0.7mm, F.Cu at (79.8, 111.1)
- added TP209: BOOT, TEST_POINT:test_point_SMD_two_pad_1mm, F.Cu at (64.5, 118.4)
- C201, C204, C205, C206, C207, C209, C215, C216, C217, C218, C219, C223, C303, C503, C603: value 100n -> 100n/16V
- C202, C203, C208, C210, C220, C307, C508, C607: value 10u -> 10u/10V
- C211, C212: value 3p3 -> 3p3/50V
- C213, C214: value 12p -> 12p/50V
- C221, C222: value 20p -> 20p/16V
- C301, C501, C601: value 47n -> 47n/25V
- C302, C305, C306, C502, C506, C507, C602, C605, C606: value 1u -> 1u/25V
- C304, C308, C401, C403, C404, C504, C505, C604, C608: value 10u -> 10u/25V
- C402: value 3.3n -> 3.3n/25V
- D401: value 3V3 -> 3V3_G
- D402: value VIN -> VIN_G
- J202: value Molex_0530470810 -> AMPHENOL_75869-132LF; footprint Molex_0530470810:MOLEX_0530470810 -> AMPHENOL_75869-132LF:AMPHENOL_75869-132LF
- J203: value SWD -> STM32_SWD; footprint A1001WV-S-6P:A1001WV-S-6P -> PogoPin:PogoConnector
- moved J202 27.9 mm to (89.0, 114.4), turned to -90 degrees
- moved R403 8.19 mm to (30.4, 96.5), turned to 0 degrees
- moved R401 8.15 mm to (30.5, 94.9), turned to 0 degrees
- moved R409 4.14 mm to (45.0, 100.8), turned to 180 degrees
- moved R208 4.03 mm to (40.6, 95.8), turned to 90 degrees
- moved Q402 3.59 mm to (40.7, 107.3), turned to 90 degrees
- moved R408 3.02 mm to (45.0, 104.0), turned to 180 degrees
- moved D402 2.69 mm to (33.0, 96.5), turned to 180 degrees
- moved D401 2.62 mm to (33.0, 94.9), turned to 180 degrees
- moved R209 2.56 mm to (41.7, 95.8), turned to 90 degrees
- moved Q401 2.37 mm to (40.7, 102.2), turned to 90 degrees
- moved J203 2.31 mm to (69.3, 88.6), turned to 0 degrees
- moved R407 1.75 mm to (45.0, 101.9), turned to 0 degrees
- moved C401 0.94 mm to (41.6, 112.9)
- moved R406 0.64 mm to (45.0, 103.0), turned to 0 degrees
Connections:
- net /MCU/ESP_CHIP_EN renamed ESP_CHIP_EN
- net ESP_INTER_ACC renamed ESP_INT2_ACC
- C216 pad 1: ESP_INTER_GYR/BOOT -> ESP_BOOT
- C223 pad 1: DRVR_DRVOFF/NRST -> STM_NRST
- J202 pad 8: ESP_INTER_GYR/BOOT -> ESP_INT1_GYR
- J203 pad 5: DRVR_DRVOFF/NRST -> STM_NRST
- R210 pad 1: ESP_INTER_GYR/BOOT -> ESP_BOOT
- R304 pad 1: +3V3 -> AVDD
- R504 pad 1: +3V3 -> AVDD
- R604 pad 1: +3V3 -> AVDD
- SW202 pad 2: ESP_INTER_GYR/BOOT -> ESP_BOOT
- U201 pad 2: /MCU/ESP_SPI_DI -> /MCU/ESP_SPI_DO
- U201 pad 5: /MCU/ESP_SPI_CLK -> /MCU/ESP_SPI_DI
- U201 pad 6: /MCU/ESP_SPI_DO -> /MCU/ESP_SPI_CLK
- U202 pad 15: ESP_INTER_GYR/BOOT -> ESP_BOOT
- U202 pad 16: ESP_GPIO10 -> /MCU/ESP_STAT
- U202 pad 27: ESP_UART_RX -> unconnected-(U202-U0RXD-Pad27)
- U202 pad 28: ESP_UART_TX -> unconnected-(U202-U0TXD-Pad28)
- U202 pad 5: /MCU/ESP_GPIO1 -> ESP_INT1_GYR
- U204 pad 11: ESP_FSPI_D -> ESP_FSPI_Q
- U204 pad 12: ESP_FSPI_Q -> ESP_FSPI_D
- U204 pad 20: DRVP_DRVOFF -> DRVP_ALARM
- U204 pad 25: DRVY_DRVOFF -> /MCU/STM_STAT
- U204 pad 31: DRVP_ALARM -> Net-(U204-PB8-BOOT0)
- U204 pad 4: DRVR_DRVOFF/NRST -> STM_NRST
- U301 pad 21: DRVY_DRVOFF -> GND
- U301 pad 27: unconnected-(U301A-AVDD-Pad27) -> AVDD
- U301 pad 29: unconnected-(U301A-FG-Pad29) -> Net-(U301A-FG)
- U501 pad 21: DRVP_DRVOFF -> GND
- U501 pad 27: unconnected-(U501A-AVDD-Pad27) -> AVDD
- U501 pad 29: unconnected-(U501A-FG-Pad29) -> Net-(U501A-FG)
- U601 pad 21: DRVR_DRVOFF/NRST -> GND
- U601 pad 27: unconnected-(U601A-AVDD-Pad27) -> AVDD
- U601 pad 29: unconnected-(U601A-FG-Pad29) -> Net-(U601A-FG)
Routing:
- net AVDD: track 0.00 -> 66.1 mm, vias 0 -> 6
- net DRVR_DRVOFF/NRST: track 64.0 -> 0.00 mm, vias 6 -> 0
- net /MCU/ESP_STAT: track 0.00 -> 48.4 mm, vias 0 -> 4
- net DRVP_DRVOFF: track 43.9 -> 0.00 mm, vias 4 -> 0
- net ESP_INT1_GYR: track 0.00 -> 43.7 mm, vias 0 -> 2
- net +3V3: track 194.4 -> 153.4 mm, vias 35 -> 33
- net STM_NRST: track 0.00 -> 40.1 mm, vias 0 -> 4
- net /MCU/STM_STAT: track 0.00 -> 33.9 mm, vias 0 -> 2
- net ESP_INT2_ACC: track 10.4 -> 41.0 mm, vias 1 -> 2
- net DRVY_DRVOFF: track 30.1 -> 0.00 mm, vias 4 -> 0
- net ESP_IMU_NCS: track 12.3 -> 41.8 mm, vias 1 -> 2
- net ESP_INTER_GYR/BOOT: track 29.2 -> 0.00 mm, vias 2 -> 0
- net ESP_BOOT: track 0.00 -> 24.0 mm, vias 0 -> 2
- net VBUS: track 21.6 -> 8.44 mm, vias 11 -> 9
- net ESP_FSPI_CLK: track 32.5 -> 44.7 mm, vias 2 -> 3
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- added copper zone on F.Cu, net VSYS
Other:
- board text added: "3V3"
- board text added: "STAT1"
- board text added: "STAT2"
- board text added: "SynchGaze Motor Control rev 1.1 12.24"
- board text added: "VIN"
- board text removed: "SynchGaze Motor Control rev 1.0 21.09.24"
