File: SynchGaze_Transmiter/MCU.kicad_sch (KiCad schematic)
At the start: 42 parts, among them J201 12401948E412A, J202 Molex_0530470810, SW201 EN, SW202 BOOT, U201 ESP32C3, U202 W25Q16JVZPIQ, U203 USBLC6-2SC6, U204 LSM6DSMTR, X201 XRCGB40M000F4M02R0

Commit message: rev 1.1
Parts:
- removed J201: 12401948E412A, USBC20_12401948E412A:AMPHENOL_12401948E412A, symbol 12401948E412A:12401948E412A
- removed J202: Molex_0530470810, Molex_0530470810:MOLEX_0530470810, symbol Connector_Generic:Conn_01x08
- removed R209: 470R, Resistor_SMD:R_0402_1005Metric, symbol Device:R_Small
- added D201: STATUS_Y, LED_SMD:LED_0603_1608Metric, symbol Device:LED
- added J201: USB4105-GF-A, USB4105-GF-A:GCT_USB4105-GF-A, symbol USB4105-GF-A:USB4105-GF-A
- added R211, R213: 5k1, Resistor_SMD:R_0402_1005Metric, symbol Device:R_Small
- added TP201: INT2_ACC_TP, TEST_POINT:test_point_SMD_0.5mm, symbol Connector:TestPoint
- added TP202: INT1_GYR_TP, TEST_POINT:test_point_SMD_0.5mm, symbol Connector:TestPoint
- added TP203: IMU_NCS_TP, TEST_POINT:test_point_SMD_0.5mm, symbol Connector:TestPoint
- added TP204: FSPI_CLK_TP, TEST_POINT:test_point_SMD_0.5mm, symbol Connector:TestPoint
- added TP205: FSPI_D_TP, TEST_POINT:test_point_SMD_0.5mm, symbol Connector:TestPoint
- added TP206: FSPI_Q_TP, TEST_POINT:test_point_SMD_0.5mm, symbol Connector:TestPoint
- added TP207, TP208, TP209: GND_TP, TEST_POINT:test_point_THT 0.7mm, symbol Connector:TestPoint
- C201, C206, C208, C212, C214: value 10u -> 10u/10V
- C202, C203, C204, C205, C207, C211, C213, C215, C216, C217: value 100n -> 100n/16V
- C209, C210: value 12p -> 12p/50V
- C218, C219: value 3p3 -> 3p3/50V
- R208: value 470R -> 1k; Manufacturer Part Number RT0402FRE07470RL -> RT0402FRE071KL; Mouser https://www.mouser.pl/ProductDetail/YAGEO/RT0402FRE07470RL?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 -> https://www.mouser.pl/ProductDetail/YAGEO/RT0402FRE071KL?qs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
Connections:
- net MCU_UART_RX is gone; now on net +3V3: R208.2
- net +3V3: now also R211.1, R213.1
- net CC1: now also J201.B5 (CC2)
- net CC2: now also J201.A5 (CC1)
- net FSPI_CLK: now also TP204.1
- net FSPI_D: now also U204.14 (SDA/SDI/SDO), TP205.1; no longer U204.1 (SDO/SA0)
- net FSPI_Q: now also U204.1 (SDO/SA0), R211.2, TP206.1; no longer U204.14 (SDA/SDI/SDO)
- net GND: now also J201.A12_B1 (GND), J201.A1_B12 (GND), TP207.1, TP208.1, TP209.1
- net GPIO10: now also D201.1 (K)
- net GPIO8: now also R213.2
- net IMU_NCS: now also TP203.1
- net SPI_CLK: now also U202.6 (CLK); no longer U202.5 (DI(IO0))
- net SPI_DI: now also U202.5 (DI(IO0)); no longer U202.2 (DO(IO1))
- net SPI_DO: now also U202.2 (DO(IO1)); no longer U202.6 (CLK)
- net USB_D+: now also J201.A6 (D1+), J201.B6 (D2+)
- net USB_D-: now also J201.A7 (D1-), J201.B7 (D2-)
- net VBUS: now also J201.A4_B9 (VBUS), J201.A9_B4 (VBUS)
- net GPIO1 renamed INT1_GYR
- net INT1_GYR: now also U204.4 (INT1), TP202.1
- net INTER_ACC renamed INT2_ACC
- net INT2_ACC: now also TP201.1
- net INTER_GYR/BOOT renamed BOOT
- net BOOT: no longer U204.4 (INT1)
- net MCU_UART_RX_R: no longer names the net of R208.1
- net MCU_UART_RX_R: now also D201.2 (A); no longer U201.27 (U0RXD)
- net MCU_UART_TX_R: no longer names the net of U201.28 (U0TXD)
- new net SHELL_GND: J201.S1 (SHELL_GND), J201.S2 (SHELL_GND), J201.S3 (SHELL_GND), J201.S4 (SHELL_GND)
- no-connect marks 7 -> 8
Other:
- moved on the sheet: C201, C202, C203, C204, C205, C206, C207, C208, C212, C213, C214, C215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
