File: SynchGaze_Transmiter/Power.kicad_sch (KiCad schematic)
At the start: 32 parts, among them U301 BQ24075TRGTR, U302 TPS63001DRCR

Commit message: rev 1.1
Parts:
- BT301: value Battery_Cell -> BAT
- C301, C303, C304, C305, C306: value 10u -> 10u/25V
- C302: value 100n -> 100n/16V; Manufacturer Part Number BQ24075TRGTR -> CL05B104JO5NNNC
- C307: value 10u -> 10u/10V
- D301: value CHRG -> CHRG_B; Manufacturer Part Number 150060BS75000 -> 150060BS55040; Mouser https://www.mouser.pl/ProductDetail/Wurth-Elektronik/150060BS75000?qs=LlUlMxKIyB2DLLpXQThavA%3D%3D -> https://www.mouser.pl/ProductDetail/Wurth-Elektronik/150060BS55040?qs=fAHHVMwC%252BbiEgEQkEQqtiA%3D%3D
- D302: value PGOOD -> PGOOD_B; Manufacturer Part Number 150060BS75000 -> 150060BS55040; Mouser https://www.mouser.pl/ProductDetail/Wurth-Elektronik/150060BS75000?qs=LlUlMxKIyB2DLLpXQThavA%3D%3D -> https://www.mouser.pl/ProductDetail/Wurth-Elektronik/150060BS55040?qs=fAHHVMwC%252BbiEgEQkEQqtiA%3D%3D
- D303: value 3V3 -> 3V3_G; Manufacturer Lite-On -> Wurth Elektronik; Manufacturer Part Number LTST-C190GKT -> 150060GS55040; Mouser https://www.mouser.pl/ProductDetail/Lite-On/LTST-C190GKT?qs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 -> https://www.mouser.pl/ProductDetail/Wurth-Elektronik/150060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
- D304: value 5V -> 5V_G; Manufacturer Lite-On -> Wurth Elektronik; Manufacturer Part Number LTST-C190GKT -> 150060GS55040; Mouser https://www.mouser.pl/ProductDetail/Lite-On/LTST-C190GKT?qs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 -> https://www.mouser.pl/ProductDetail/Wurth-Elektronik/150060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
Other:
- note removed: "Two green diodes"
- note removed: "green"
- moved on the sheet: BT301, C301, C302, C303, C304, C305, C306, C307, D301, D302, D303, D304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
