File: SynchGaze_Transmiter/SynchGaze_Transmiter.kicad_pcb (KiCad board)
At the start: 4 copper layers, 30 x 51 mm, 75 parts, among them J201 12401948E412A, J202 Molex_0530470810, SW201 EN, SW202 BOOT, U201 ESP32C3, U202 W25Q16JVZPIQ, U203 USBLC6-2SC6, U204 LSM6DSMTR, U301 BQ24075TRGTR, U302 TPS63001DRCR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

Commit message: rev 1.1
Parts:
- removed J202: Molex_0530470810, Molex_0530470810:MOLEX_0530470810
- removed R209: 470R, Resistor_SMD:R_0402_1005Metric
- added D201: STATUS_Y, LED_SMD:LED_0603_1608Metric, F.Cu at (143.5, 64.0)
- added R211: 5k1, Resistor_SMD:R_0402_1005Metric, F.Cu at (155.7, 86.4)
- added R213: 5k1, Resistor_SMD:R_0402_1005Metric, F.Cu at (155.4, 80.1)
- added TP201: INT2_ACC_TP, TEST_POINT:test_point_SMD_0.5mm, F.Cu at (157.0, 83.1)
- added TP202: INT1_GYR_TP, TEST_POINT:test_point_SMD_0.5mm, F.Cu at (158.1, 85.8)
- added TP203: IMU_NCS_TP, TEST_POINT:test_point_SMD_0.5mm, F.Cu at (161.3, 82.2)
- added TP204: FSPI_CLK_TP, TEST_POINT:test_point_SMD_0.5mm, F.Cu at (160.2, 82.2)
- added TP205: FSPI_D_TP, TEST_POINT:test_point_SMD_0.5mm, F.Cu at (159.3, 82.9)
- added TP206: FSPI_Q_TP, TEST_POINT:test_point_SMD_0.5mm, F.Cu at (157.9, 84.1)
- added TP207: GND_TP, TEST_POINT:test_point_THT 0.7mm, F.Cu at (164.5, 82.9)
- added TP208: GND_TP, TEST_POINT:test_point_THT 0.7mm, F.Cu at (156.8, 85.9)
- added TP209: GND_TP, TEST_POINT:test_point_THT 0.7mm, F.Cu at (157.8, 81.0)
- BT301: value Battery -> BAT
- C201, C206, C208, C212, C214, C307: value 10u -> 10u/10V
- C202, C203, C204, C205, C207, C211, C213, C215, C216, C217, C302: value 100n -> 100n/16V
- C209, C210: value 12p -> 12p/50V
- C218, C219: value 3p3 -> 3p3/50V
- C301, C303, C304, C305, C306: value 10u -> 10u/25V
- D301: value CHRG -> CHRG_B; footprint LED_SMD:LED_0402_1005Metric -> LED_SMD:LED_0603_1608Metric
- D302: value PGOOD -> PGOOD_B; footprint LED_SMD:LED_0402_1005Metric -> LED_SMD:LED_0603_1608Metric
- D303: value 3V3 -> 3V3_G; footprint LED_SMD:LED_0402_1005Metric -> LED_SMD:LED_0603_1608Metric
- D304: value 5V -> 5V_G; footprint LED_SMD:LED_0402_1005Metric -> LED_SMD:LED_0603_1608Metric
- J201: value 12401948E412A -> USB4105-GF-A; footprint USBC20_12401948E412A:AMPHENOL_12401948E412A -> USB4105-GF-A:GCT_USB4105-GF-A
- R208: value 470R -> 1k
- moved R208 13.8 mm to (146.1, 64.0), turned to 0 degrees
- moved J201 1.26 mm to (153.2, 51.7)
- moved R203 1.08 mm to (148.2, 61.5)
- moved R204 1.07 mm to (149.3, 61.5)
- moved U203 0.91 mm to (152.7, 62.2)
- moved C217 0.76 mm to (155.4, 79.0)
- moved R212 0.76 mm to (155.4, 77.9)
- moved R306 0.68 mm to (146.1, 57.8)
- moved D301 0.67 mm to (143.5, 57.7)
- moved R316 0.55 mm to (146.1, 60.9)
- moved R307 0.50 mm to (146.1, 59.3)
- moved D304 0.47 mm to (143.5, 60.9)
- moved C203 0.43 mm to (155.4, 76.9)
- moved D302 0.41 mm to (143.5, 59.3)
- moved SW202 0.38 mm to (141.9, 68.3)
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Connections:
- net /MCU/INTER_ACC renamed /MCU/INT2_ACC
- C217 pad 1: /MCU/INTER_GYR/BOOT -> /MCU/BOOT
- J201 pad S1: unconnected-(J201-SHELL_GND-PadS1)_0 -> SHELL_GND
- J201 pad S2: unconnected-(J201-SHELL_GND-PadS2)_0 -> SHELL_GND_0
- J201 pad S3: unconnected-(J201-SHELL_GND-PadS1) -> SHELL_GND_1
- J201 pad S4: unconnected-(J201-SHELL_GND-PadS2) -> SHELL_GND_2
- R208 pad 1: /MCU/MCU_UART_RX_R -> Net-(D201-A)
- R208 pad 2: /MCU/MCU_UART_RX -> +3V3
- R212 pad 1: /MCU/INTER_GYR/BOOT -> /MCU/BOOT
- SW202 pad 2: /MCU/INTER_GYR/BOOT -> /MCU/BOOT
- U201 pad 15: /MCU/INTER_GYR/BOOT -> /MCU/BOOT
- U201 pad 27: /MCU/MCU_UART_RX_R -> unconnected-(U201-U0RXD-Pad27)
- U201 pad 28: /MCU/MCU_UART_TX_R -> unconnected-(U201-U0TXD-Pad28)
- U201 pad 5: /MCU/GPIO1 -> /MCU/INT1_GYR
- U202 pad 2: /MCU/SPI_DI -> /MCU/SPI_DO
- U202 pad 5: /MCU/SPI_CLK -> /MCU/SPI_DI
- U202 pad 6: /MCU/SPI_DO -> /MCU/SPI_CLK
- U204 pad 1: /MCU/FSPI_D -> /MCU/FSPI_Q
- U204 pad 14: /MCU/FSPI_Q -> /MCU/FSPI_D
- U204 pad 4: /MCU/INTER_GYR/BOOT -> /MCU/INT1_GYR
Routing:
- net /MCU/INTER_GYR/BOOT: track 46.6 -> 0.00 mm, vias 4 -> 0
- net /MCU/GPIO10: track 0.00 -> 23.9 mm, vias 0 -> 2
- net /MCU/BOOT: track 0.00 -> 20.3 mm, vias 0 -> 2
- net /MCU/INT1_GYR: track 0.00 -> 11.2 mm, vias 0 -> 2
- net /MCU/CC2: track 9.26 -> 16.9 mm, vias 2 -> 0
- net /MCU/FSPI_Q: track 19.2 -> 11.8 mm, vias 2 -> 0
- net /MCU/FSPI_D: track 18.8 -> 11.7 mm, vias 3 -> 2
- net /MCU/CC1: track 6.98 -> 13.5 mm
- net GND: track 42.3 -> 36.1 mm, vias 122 -> 109
- net /MCU/IMU_NCS: track 18.3 -> 12.5 mm
- net /MCU/FSPI_CLK: track 12.1 -> 6.74 mm
- net /MCU/MCU_UART_RX_R: track 5.11 -> 0.00 mm
- net /MCU/MCU_UART_TX_R: track 4.48 -> 0.00 mm
- net +3V3: track 112.6 -> 116.8 mm, vias 16 -> 18
- net /MCU/SPI_CLK: track 6.77 -> 10.3 mm
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Other:
- outline, holes or cut-outs redrawn
- board text added: "STAT"
- board text added: "SynchGaze Transmiter rev 1.1 12.24"
- board text removed: "SynchGaze Transmiter rev 1.0 21.09.24"
